File: usb3-ngff-carrier.kicad_pcb (KiCad board)
At the start: 4 copper layers, 90 x 40 mm, 60 parts, among them J1 692221030100, J2 2199119-3, J3 Jack-DC, J4 SIM8060-6-1-14-00-A, J5 Conn_01x03_Male, J6 SIM8060-6-1-14-00-A, SW1 KMR221GLFS, U1 AP62301WU7

Commit message: Add: Issue B changes finalised
Parts:
- added R13: 10k, Resistor_SMD:R_0603_1608Metric, B.Cu at (33.1, 20.9)
- added R14: 10k, Resistor_SMD:R_0603_1608Metric, B.Cu at (47.1, 21.6)
- J1: value 692221030100 -> KUSBX-BS1N9-1-BL30
- L1: value 3.3uH -> 2.2uH
- moved TP4 0.49 mm to (30.3, 24.9)
- moved C11 0.25 mm to (32.1, 34.6)
- moved C15 0.25 mm to (12.2, 4.25)
- moved C3 0.25 mm to (8.50, 4.25)
- moved C5 0.25 mm to (29.9, 5.40)
- moved C6 0.25 mm to (32.1, 5.40)
- moved C10 0.15 mm to (29.8, 34.6)
- moved C23 0.10 mm to (34.1, 23.4)
Connections:
- J2 pad 29: /USB_SS_RX_N -> /USB_SS_TX_N
- J2 pad 31: /USB_SS_RX_P -> /USB_SS_TX_P
- J2 pad 35: /USB_SS_TX_N -> /USB_SS_RX_N
- J2 pad 37: /USB_SS_TX_P -> /USB_SS_RX_P
Routing:
- net GND: track 41.7 -> 56.3 mm, vias 342 -> 337
- net /USIM2_VDD: track 43.8 -> 50.6 mm
- net /USIM1_VDD: track 24.8 -> 27.5 mm
- net Net-(C23-Pad1): track 3.15 -> 4.77 mm
- net /USIM1_DATA: track 2.88 -> 4.46 mm
- net Net-(C19-Pad1): track 3.15 -> 4.72 mm
- net /SW: track 6.55 -> 5.11 mm
- net /USIM1_RST: track 9.27 -> 8.21 mm
- net /WAKE_ON_WAN: track 5.44 -> 6.22 mm
- net /USB_SS_TX_P: track 22.0 -> 22.7 mm
- net /USB_SS_TX_N: track 22.0 -> 22.7 mm
- net /USIM1_CLK: track 6.38 -> 6.94 mm
- net VSYS: track 5.49 -> 5.24 mm, vias 14 -> 15
