File: usb3-ngff-carrier.sch (KiCad schematic (older format))
At the start: 53 parts, among them J1 KUSBX-BS1N9-1-BL30, J2 2199119-3, J3 Jack-DC, J4 SIM8060-6-1-14-00-A, J5 Conn_01x03_Male, J6 SIM8060-6-1-14-00-A, SW1 KMR221GLFS, U1 AP62301WU7

Commit message: Add: Issue B changes finalised
Parts:
- added R13, R14: 10k, Resistor_SMD:R_0603_1608Metric, symbol Device:R_Small
- C15, C3: Int @ 10 0.386 -> 0.248; MPN TMK325B7226MMHP -> CL32B226MOJNNNE; Mfr Taiyo-Yuden -> Samsung Electro-Mechanics; SKU 963-TMK325B7226MMHP -> 187-CL32B226MOJNNNE
- J4, J6: footprint GCT_SIM8060-6-1-14-00-A -> footprint:GCT_SIM8060-6-1-14-00-A
Connections:
- net USB_SS_RX_N: now also J2.35; no longer J2.29
- net USB_SS_RX_P: now also J2.37; no longer J2.31
- net USB_SS_TX_N: now also J2.29; no longer J2.35
- net USB_SS_TX_P: now also J2.31; no longer J2.37
- net USIM1_VDD: now also R13.1
- net USIM2_VDD: now also R14.1
- net at C23.1, J4.C7 (IO), R12.1: now also R13.2
- net at C19.1, J6.C7 (IO), R8.1: now also R14.2
Other:
- note added: "Some modules (RM500Q-GL) have the USB SS\nAC-coupling capacitors integrated. They are\nNOT present on this design for this reason.\n\nSome modules may require them. CHECK."
- note removed: "Some modules (RM500Q-GL) have the USB SS\nAC-coupling capacitors integrated. They are\nNOT present on this design for this reason.\n\nSome modules may require them. CHECK.\n\nADDITIONALLY - Note that the TX-RX pairing flips here."
